File: ElectronicTriggerUnit_PCB_Files/ElectronicTriggerUnit.kicad_sch (KiCad schematic)
At the start: 51 parts, among them IC1 MCP1407-E_SN, IC2 ATTINY814-SSF, J2 Conn_01x05, J4 Conn_01x04, M1 Motor_DC, Q1 LC191PTDT, Q2 LKPT30102B-A01, Q3 78-SQRS140ELP, Q4 LC191PTDT, U1 Gnd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

Commit message: Fixes
Parts:
- C1, C12: footprint Capacitor_THT:C_Axial_L5.1mm_D3.1mm_P7.50mm_Horizontal -> Capacitor_SMD:C_0603_1608Metric
Changed lines of the file:
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@@
 			)
 		)
-		(property "Footprint" "Capacitor_THT:C_Axial_L5.1mm_D3.1mm_P7.50mm_Horizontal"
+		(property "Footprint" "Capacitor_SMD:C_0603_1608Metric"
 			(at 183.8452 59.69 0)
 			(effects
@@
 			)
 		)
-		(property "Footprint" "Capacitor_THT:C_Axial_L5.1mm_D3.1mm_P7.50mm_Horizontal"
+		(property "Footprint" "Capacitor_SMD:C_0603_1608Metric"
 			(at 193.3448 52.07 0)
 			(effects

Commit message: Fixes
Parts:
- C1, C12: footprint Capacitor_SMD:C_0603_1608Metric -> Capacitor_THT:C_Axial_L5.1mm_D3.1mm_P7.50mm_Horizontal
Changed lines of the file:
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@@
 			)
 		)
-		(property "Footprint" "Capacitor_SMD:C_0603_1608Metric"
+		(property "Footprint" "Capacitor_THT:C_Axial_L5.1mm_D3.1mm_P7.50mm_Horizontal"
 			(at 183.8452 59.69 0)
 			(effects
@@
 			)
 		)
-		(property "Footprint" "Capacitor_SMD:C_0603_1608Metric"
+		(property "Footprint" "Capacitor_THT:C_Axial_L5.1mm_D3.1mm_P7.50mm_Horizontal"
 			(at 193.3448 52.07 0)
 			(effects
