File: ElectronicTriggerUnit_PCB_Files/ElectronicTriggerUnit.kicad_pcb (KiCad board)
At the start: 2 copper layers, 59.7 x 50 mm, 50 parts, among them IC1 MCP1407-E_SN, IC2 ATTINY814-SSF, J2 Conn_01x05, J4 Conn_01x04, Q1 LC191PTDT, Q2 LKPT30102B-A01, Q3 78-SQRS140ELP, Q4 LC191PTDT, U1 Gnd, U2 12v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

Commit message: changed some parts
Parts:
- removed D4: D, Diode_SMD:D_0603_1608Metric
- added IC3: BU4S584G2-TR, SamacSys:SOT95P280X125-5N, F.Cu at (79.3, 116.5)
- R4: footprint Resistor_SMD:R_0603_1608Metric -> Resistor_SMD:R_1206_3216Metric
- moved R14 25.3 mm to (101.4, 118.6), turned to 90 degrees
- moved R13 9.16 mm to (86.9, 116.4), turned to 180 degrees
- moved C11 8.37 mm to (86.8, 117.9)
- moved R1 8.32 mm to (105.8, 82.9), turned to -90 degrees
- moved R4 4.39 mm to (109.8, 91.9), turned to 180 degrees
- moved C1 4.15 mm to (105.4, 92.2), turned to 180 degrees
- moved C12 3.61 mm to (105.4, 90.7), turned to 0 degrees
- moved U3 3.05 mm to (123.0, 87.3)
- moved D2 2.30 mm to (121.0, 93.0)
- moved Q3 2.12 mm to (118.3, 87.2)
- moved IC1 1.87 mm to (108.8, 87.2), turned to 0 degrees
- moved U1 1.85 mm to (116.3, 81.8)
- moved U5 1.85 mm to (116.3, 92.8)
- moved C8 1.31 mm to (82.7, 84.6)
- moved C9 1.31 mm to (81.2, 84.6)
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Connections:
- net /trigger_Out renamed Net-(IC3-A)
- IC1 pad 7: unconnected-(IC1-OUT_2-Pad7) -> GND
- IC1 pad 8: unconnected-(IC1-VDD_2-Pad8) -> GND
- LED4 pad 3: GND -> (no net)
- Q2 pad 3: GND -> (no net)
Routing:
- net /trigger_Out: track 0.00 -> 11.2 mm
- net Net-(S1-NO): track 23.7 -> 14.9 mm
- net /NMOS: track 22.1 -> 28.1 mm
- net +12V: track 73.7 -> 79.6 mm, vias 0 -> 1
- net +3.3V: track 87.2 -> 82.4 mm
- net GND: track 56.3 -> 51.9 mm, vias 12 -> 13
- net Net-(Q3-Pad4): track 1.90 -> 5.79 mm
- net /Semi_Auto: track 41.3 -> 38.8 mm
- net /V_Cycle_In: track 9.40 -> 8.77 mm
- net /updiRx: track 13.2 -> 13.8 mm
- net Net-(LED1-Pad2): track 6.80 -> 7.32 mm
- net /pwr_motor: vias 0 -> 1
Other:
- board size 59.7 x 50 mm -> 61.3 x 50 mm
