File: ElectronicTriggerUnit_PCB_Files/ElectronicTriggerUnit.kicad_pcb (KiCad board)
At the start: 2 copper layers, 61.3 x 79 mm, 59 parts, among them IC1 MCP1407-E_SN, IC2 ATTINY814-SSF, IC3 BU4S584G2-TR, IC4 MCP1407-E_SN, J2 Conn_01x05, J4 Conn_01x04, Q1 LC191PTDT, Q2 LKPT30102B-A01, Q3 SIR500DP-T1-RE3, Q4 LC191PTDT, Q5 SIR500DP-T1-RE3, U1 Gnd, U2 12v, U3 GndMotor, U4 Gnd, U5 12v, U6 12v, U7 Gnd, U8 SigIn

Commit message: added a different combo
Parts:
- removed the LED2 at (102.2, 102.2)
- removed the Q4 at (106.7, 102.2)
- added C16: 10n, Capacitor_SMD:C_0603_1608Metric, F.Cu at (166.4, 128.8)
- added C17: 10n, Capacitor_SMD:C_0603_1608Metric, F.Cu at (137.6, 122.9)
- added C18: 1u, Capacitor_SMD:C_0603_1608Metric, F.Cu at (165.6, 112.1)
- added C19: 10n, Capacitor_SMD:C_0603_1608Metric, F.Cu at (167.1, 112.1)
- added C20: 10u/1206, Capacitor_SMD:C_0603_1608Metric, F.Cu at (141.3, 128.8)
- added C21: 10u/1206, Capacitor_SMD:C_0603_1608Metric, F.Cu at (141.3, 130.1)
- added C22: 22n, Capacitor_SMD:C_0603_1608Metric, F.Cu at (143.1, 126.1)
- added C23: 22u, Capacitor_SMD:C_0603_1608Metric, F.Cu at (139.9, 121.3)
- added C24: 22u, Capacitor_SMD:C_0603_1608Metric, F.Cu at (141.4, 121.3)
- added C25: 100p, Capacitor_SMD:C_0603_1608Metric, F.Cu at (144.4, 121.3)
- added C26: 100nf, Capacitor_SMD:C_0603_1608Metric, F.Cu at (167.2, 122.0)
- added D4: B340A, Diode_SMD:D_SMA, F.Cu at (149.7, 129.0)
- added IC5: ATTINY814-SSF, SamacSys:SOIC127P600X175-14N, F.Cu at (160.0, 114.0)
- added IC6: BU4S584G2-TR, SamacSys:SOT95P280X125-5N, F.Cu at (170.9, 123.5)
- added J3: Conn_01x04, Connector_PinHeader_2.54mm:PinHeader_1x04_P2.54mm_Vertical, F.Cu at (164.6, 108.6)
- added L2: 10u/C2921170, Inductor_SMD:L_Chilisin_BMRA00040420, F.Cu at (149.0, 122.6)
- added LED3: LKIR30102C-A01, SamacSys:APA3010P3C, F.Cu at (139.4, 108.6)
- added LED4: XL-2012IRC-940, SamacSys:LEDC2012X105N, B.Cu at (165.5, 131.5)
- added PS2: AP5100WG-7, SamacSys:SOT95P285X140-6N, F.Cu at (140.5, 126.1)
- added Q5: LC191PTDT, SamacSys:AP1608P1CP22, B.Cu at (165.5, 127.2)
- added Q6: LKPT30102B-A01, SamacSys:APA3010P3C, F.Cu at (134.2, 121.2)
- added R17: 5K, Resistor_SMD:R_0603_1608Metric, F.Cu at (138.3, 120.2)
- added R18: 5K, Resistor_SMD:R_0603_1608Metric, F.Cu at (167.2, 126.5)
- added R19: 100R, Resistor_SMD:R_0603_1608Metric, F.Cu at (142.6, 110.4)
- added R20: 100R, Resistor_SMD:R_0603_1608Metric, F.Cu at (168.0, 128.7)
- added R21: 10k, Resistor_SMD:R_0603_1608Metric, F.Cu at (168.6, 112.1)
- added R22: 1k, Resistor_SMD:R_0603_1608Metric, F.Cu at (171.0, 111.2)
- added R23: 10k, Resistor_SMD:R_0603_1608Metric, F.Cu at (138.0, 128.2)
- added R24: 2k, Resistor_SMD:R_0603_1608Metric, F.Cu at (136.4, 126.6)
- added R25: 10k, Resistor_SMD:R_0603_1608Metric, F.Cu at (145.9, 121.3)
- added R26: 3.3k, Resistor_SMD:R_0603_1608Metric, F.Cu at (142.9, 122.9)
- added R27: 10K, Resistor_SMD:R_0603_1608Metric, F.Cu at (167.2, 125.0)
- added R28: 1K, Resistor_SMD:R_0603_1608Metric, F.Cu at (167.2, 123.5)
- added S2: Trigger, SamacSys:463092691402, F.Cu at (163.7, 119.9)
- added U10: Gnd, SamacSys:Copper_Pad, F.Cu at (146.3, 131.1)
- added U11: GndMotor, SamacSys:Copper_Pad, F.Cu at (141.3, 134.2)
- added U9: 12v, SamacSys:Copper_Pad, F.Cu at (141.3, 132.0)
- R1: renamed from R5; value 10k -> 5K
- R2: renamed from R3; value 10k -> 5K
- R3: renamed from R6; value 51R -> 100R
- R4: renamed from R10; value 91R -> 100R
- moved C7 84.0 mm to (156.8, 97.2)
- moved Q4 84.0 mm to (144.3, 101.3)
- moved U6 84.0 mm to (151.7, 82.1)
- moved R10 84.0 mm to (152.0, 97.7)
- moved R9 84.0 mm to (155.2, 87.0)
- moved U8 84.0 mm to (149.8, 101.9)
- moved D2 84.0 mm to (135.6, 97.4)
- moved IC3 84.0 mm to (155.4, 91.5)
- moved C8 83.3 mm to (155.1, 97.4)
- moved U7 83.3 mm to (152.4, 85.1)
- renumbered C13 to C1, C5 to C10, C7 to C11, C9 to C12, C8 to C13, C10 to C14, C11 to C15, C4 to C2, C2 to C3, C3 to C4, C12 to C5, C1 to C6, C14 to C7, C15 to C8, C6 to C9, D2 to D1, D3 to D2, D1 to D3, IC2 to IC1, IC1 to IC2, IC4 to IC3, IC3 to IC4, J4 to J1, LED4 to LED1, LED1 to LED2, Q5 to Q4, R15 to R10, R7 to R11, R8 to R12, R9 to R13, R12 to R14, R14 to R15, R13 to R16, R2 to R5, R11 to R6, R1 to R7, R4 to R8, R16 to R9, U5 to U1, U1 to U5, U8 to U7, U7 to U8
Connections:
- net /NMOS renamed /ControlSensorCombo/NMOS
- net /Semi_Auto renamed /ControlSensorCombo/Semi_Auto
- net /Semi_Auto_In renamed /ControlSensorCombo/Semi_Auto_In
- net /V_Cycle_In renamed /ControlSensorCombo/V_Cycle_In
- net /V_Cycle_Out renamed /ControlSensorCombo/V_Cycle_Out
- net /V_FB renamed /ControlSensorCombo/BuckStepDown/V_FB
- net /pwr_motor renamed /ControlSensorCombo/pwr_motor
- net /pwr_motor_ring renamed /SensorRingCombo/pwr_motor_ring
- net /sigIn renamed /SensorRingCombo/sigIn
- net /trigger_In renamed /ControlSensorCombo/trigger_In
- net /trigger_Out renamed /ControlSensorCombo/trigger_Out
- net /updiRx renamed /ControlSensorCombo/updiRx
- net /updiTx renamed /ControlSensorCombo/updiTx
- IC3 pad 6: Net-(IC4-OUT_1) -> Net-(IC3-OUT_1)
- IC3 pad 7: unconnected-(IC4-OUT_2-Pad7) -> Net-(IC3-OUT_1)
- R10 pad 2: Net-(IC4-OUT_1) -> Net-(IC3-OUT_1)
Routing:
- net +3.3V: track 81.5 -> 161.3 mm, vias 0 -> 2
- net /SensorRingCombo/V_Cycle: track 0.00 -> 40.8 mm, vias 0 -> 2
- net /SensorRingCombo/sigOut: track 0.00 -> 38.3 mm, vias 0 -> 2
- net /SensorRingCombo/Semi_Auto: track 0.00 -> 23.1 mm, vias 0 -> 1
- net /SensorRingCombo/updiRx: track 0.00 -> 21.3 mm
- net /SensorRingCombo/trigger: track 0.00 -> 17.3 mm
- net Net-(D4-K): track 0.00 -> 11.6 mm
- net +12V: track 123.6 -> 132.6 mm
- net Net-(LED4-Pad2): track 0.00 -> 8.68 mm, vias 0 -> 1
- net /SensorRingCombo/BuckStepDown1/V_FB: track 0.00 -> 8.62 mm
- net Net-(IC6-A): track 0.00 -> 5.78 mm
- net Net-(IC3-OUT_1): track 0.00 -> 5.34 mm
- net Net-(S2-NO): track 0.00 -> 4.16 mm
- net Net-(IC4-OUT_1): track 3.30 -> 0.00 mm
- net Net-(PS2-EN): track 0.00 -> 3.18 mm
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Other:
- board size 61.3 x 79 mm -> 109.6 x 57.2 mm
- board text added: "Control and Sensor Combo"
- board text added: "Sensor and Ring Combo"

Commit message: small fixes for new combo
Parts:
- moved U11 27.0 mm to (154.2, 110.5), turned to 90 degrees
- moved R24 13.5 mm to (149.8, 128.0), turned to 90 degrees
- moved D4 13.3 mm to (151.5, 115.8), turned to 90 degrees
- moved C21 13.0 mm to (151.4, 122.0), turned to 90 degrees
- moved R23 12.2 mm to (149.8, 125.0), turned to 90 degrees
- moved U9 12.1 mm to (152.0, 126.3), turned to 90 degrees
- moved C24 11.9 mm to (148.2, 111.5), turned to 0 degrees
- moved C23 11.7 mm to (148.2, 113.0), turned to 0 degrees
- moved C20 10.9 mm to (149.8, 122.0), turned to 90 degrees
- moved PS2 7.20 mm to (146.9, 122.8), turned to 0 degrees
- moved C22 7.00 mm to (146.9, 120.2), turned to 0 degrees
- moved L2 6.21 mm to (147.4, 116.6)
- moved R25 6.16 mm to (140.2, 123.8), turned to 0 degrees
- moved U10 4.97 mm to (142.5, 127.9), turned to -90 degrees
- moved C25 4.20 mm to (140.3, 122.2), turned to 0 degrees
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Connections:
- J3 pad 3: /SensorRingCombo/updiRx -> /SensorRingCombo/updiTx
- J3 pad 4: /SensorRingCombo/updiTx -> /SensorRingCombo/updiRx
Routing:
- net /SensorRingCombo/sigOut: track 38.3 -> 8.17 mm, vias 2 -> 0
- net +12V: track 132.6 -> 107.9 mm, vias 1 -> 2
- net +3.3V: track 161.3 -> 183.6 mm
- net GND: track 60.0 -> 71.0 mm, vias 20 -> 25
- net /SensorRingCombo/pwr_motor_ring: track 3.80 -> 7.60 mm, vias 0 -> 1
- net Net-(D4-K): track 11.6 -> 8.10 mm
- net /SensorRingCombo/BuckStepDown1/V_FB: track 8.62 -> 6.03 mm
- net Net-(LED3-Pad1): track 0.00 -> 1.81 mm
- net /SensorRingCombo/V_Cycle: track 40.8 -> 39.2 mm
- net /SensorRingCombo/updiRx: track 21.3 -> 22.9 mm
- net Net-(PS2-EN): track 3.18 -> 4.13 mm
