File: ElectronicTriggerUnit_PCB_Files/sensor_ring.kicad_sch (KiCad schematic)
At the start: 24 parts, among them IC5 ATTINY814-SSF, J3 Conn_01x04, M2 Motor_DC, Q5 LC191PTDT, Q6 LKPT30102B-A01, U10 Gnd, U11 GndMotor, U6 12v, U7 SigIn, U8 Gnd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

Commit message: small fixes for new combo
Connections:
- net updiRx: now also J3.4 (Pin_4); no longer J3.3 (Pin_3)
- net updiTx: now also J3.3 (Pin_3); no longer J3.4 (Pin_4)
Changed lines of the file:
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@@
 	)
 	(label "updiRx"
-		(at 156.21 161.29 180)
+		(at 156.21 163.83 180)
 		(fields_autoplaced yes)
 		(effects
@@
 	)
 	(label "updiTx"
-		(at 156.21 163.83 180)
+		(at 156.21 161.29 180)
 		(fields_autoplaced yes)
 		(effects
