File: PCB_Files/ElectronicTriggerUnit.kicad_sch (KiCad schematic)
At the start: 0 parts

Commit message: moved to platformio
Other:
- added sheet NormalEtu (normal_etu.kicad_sch)
Changed lines of the file:
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@@
 (kicad_sch
-	(version 20231120)
+	(version 20250114)
 	(generator "eeschema")
-	(generator_version "8.0")
+	(generator_version "9.0")
 	(paper "A4")
 	(text "R12 = (R9 * 0.81) / (Vo - 0.81)"
@@
 		(at 58.42 59.69)
 		(size 43.18 29.21)
+		(exclude_from_sim no)
+		(in_bom yes)
+		(on_board yes)
+		(dnp no)
 		(fields_autoplaced yes)
 		(stroke
@@
 	)
 	(sheet
-		(at 163.83 59.69)
+		(at 147.32 59.69)
+		(size 48.26 29.21)
+		(exclude_from_sim no)
+		(in_bom yes)
+		(on_board yes)
+		(dnp no)
+		(fields_autoplaced yes)
+		(stroke
+			(width 0.1524)
+			(type solid)
+		)
+		(fill
+			(color 0 0 0 0.0000)
+		)
+		(property "Sheetname" "NormalEtu"
+			(at 147.32 58.9784 0)
+			(effects
+				(font
+					(size 1.27 1.27)
+				)
+				(justify left bottom)
+			)
+		)
+		(property "Sheetfile" "normal_etu.kicad_sch"
+			(at 147.32 89.4846 0)
+			(effects
+				(font
+					(size 1.27 1.27)
+				)
+				(justify left top)
+			)
+		)
+		(instances
+			(project "ElectronicTriggerUnit"
+				(path "/006bc43b-d3a8-4a38-a8dc-5a24da3f9b4d"
+					(page "10")
+				)
+			)
+		)
+	)
+	(sheet
+		(at 102.87 59.69)
 		(size 43.18 29.21)
+		(exclude_from_sim no)
+		(in_bom yes)
+		(on_board yes)
+		(dnp no)
 		(fields_autoplaced yes)
 		(stroke
@@
 		)
 		(property "Sheetname" "SensorRingCombo"
-			(at 163.83 58.9784 0)
+			(at 102.87 58.9784 0)
 			(effects
 				(font
@@
 		)
 		(property "Sheetfile" "sensor_ring.kicad_sch"
-			(at 163.83 89.4846 0)
+			(at 102.87 89.4846 0)
 			(effects
 				(font
@@
 		)
 	)
+	(embedded_fonts no)
 )

Commit message: stacked version
Other:
- added sheet LayeredEtu (layered_etu.kicad_sch)
Changed lines of the file:
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@@
+		)
+	)
+	(sheet
+		(at 198.12 59.69)
+		(size 38.1 29.21)
+		(exclude_from_sim no)
+		(in_bom yes)
+		(on_board yes)
+		(dnp no)
+		(fields_autoplaced yes)
+		(stroke
+			(width 0.1524)
+			(type solid)
+		)
+		(fill
+			(color 0 0 0 0.0000)
+		)
+		(property "Sheetname" "LayeredEtu"
+			(at 198.12 58.9784 0)
+			(effects
+				(font
+					(size 1.27 1.27)
+				)
+				(justify left bottom)
+			)
+		)
+		(property "Sheetfile" "layered_etu.kicad_sch"
+			(at 198.12 89.4846 0)
+			(effects
+				(font
+					(size 1.27 1.27)
+				)
+				(justify left top)
+			)
+		)
+		(instances
+			(project "ElectronicTriggerUnit"
+				(path "/006bc43b-d3a8-4a38-a8dc-5a24da3f9b4d"
+					(page "14")
+				)
+			)
 		)
 	)
