File: PCB_Files/buck.kicad_sch (KiCad schematic)
At the start: 13 parts

Commit message: moved to platformio
Parts:
- renumbered C9 to C20, C10 to C21, C11 to C22, C12 to C23, C13 to C24, C14 to C25, D3 to D4, L1 to L2, PS1 to PS2, R11 to R23, R12 to R24, R13 to R25, R14 to R26
Changed lines of the file:
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@@
 (kicad_sch
-	(version 20231120)
+	(version 20250114)
 	(generator "eeschema")
-	(generator_version "8.0")
+	(generator_version "9.0")
 	(paper "A4")
 	(junction
@@
 	(label "V_FB"
 		(at 157.48 92.71 180)
-		(fields_autoplaced yes)
 		(effects
 			(font
@@
 	(label "V_FB"
 		(at 196.85 97.79 180)
-		(fields_autoplaced yes)
 		(effects
 			(font
@@
 		(shape output)
 		(at 99.06 52.07 180)
-		(fields_autoplaced yes)
 		(effects
 			(font
@@
 		(shape input)
 		(at 99.06 48.26 180)
-		(fields_autoplaced yes)
 		(effects
 			(font
@@
 		(shape input)
 		(at 99.06 55.88 180)
-		(fields_autoplaced yes)
 		(effects
 			(font
@@
 		(dnp no)
 		(fields_autoplaced yes)
-		(property "Reference" "R13"
+		(property "Reference" "R25"
 			(at 187.96 90.1699 0)
 			(effects
@@
 				(path "/006bc43b-d3a8-4a38-a8dc-5a24da3f9b4d/539d63da-e1ff-4f16-be2c-1db8c9db8078/6918b752-c4f8-49c7-b2f5-91fa140447ec"
 					(reference "R13")
+					(unit 1)
+				)
+				(path "/006bc43b-d3a8-4a38-a8dc-5a24da3f9b4d/567dbb32-3fa8-4c8f-b406-7d7df1e784be/a9023d18-0b2d-43c7-9654-aa2d0b287c66"
+					(reference "R39")
 					(unit 1)
 				)
@@
 		(dnp no)
 		(fields_autoplaced yes)
-		(property "Reference" "R12"
+		(property "Reference" "R24"
 			(at 120.65 102.8699 0)
 			(effects
@@
 				(path "/006bc43b-d3a8-4a38-a8dc-5a24da3f9b4d/539d63da-e1ff-4f16-be2c-1db8c9db8078/6918b752-c4f8-49c7-b2f5-91fa140447ec"
 					(reference "R12")
+					(unit 1)
+				)
+				(path "/006bc43b-d3a8-4a38-a8dc-5a24da3f9b4d/567dbb32-3fa8-4c8f-b406-7d7df1e784be/a9023d18-0b2d-43c7-9654-aa2d0b287c66"
+					(reference "R38")
 					(unit 1)
 				)
@@
 		(dnp no)
 		(fields_autoplaced yes)
-		(property "Reference" "C14"
+		(property "Reference" "C25"
 			(at 201.041 92.0663 0)
 			(effects
@@
 				(path "/006bc43b-d3a8-4a38-a8dc-5a24da3f9b4d/539d63da-e1ff-4f16-be2c-1db8c9db8078/6918b752-c4f8-49c7-b2f5-91fa140447ec"
 					(reference "C14")
+					(unit 1)
+				)
+				(path "/006bc43b-d3a8-4a38-a8dc-5a24da3f9b4d/567dbb32-3fa8-4c8f-b406-7d7df1e784be/a9023d18-0b2d-43c7-9654-aa2d0b287c66"
+					(reference "C37")
 					(unit 1)
 				)
@@
 		(dnp no)
 		(fields_autoplaced yes)
-		(property "Reference" "C9"
+		(property "Reference" "C20"
 			(at 103.251 93.3363 0)
 			(effects
@@
 				(path "/006bc43b-d3a8-4a38-a8dc-5a24da3f9b4d/539d63da-e1ff-4f16-be2c-1db8c9db8078/6918b752-c4f8-49c7-b2f5-91fa140447ec"
 					(reference "C9")
+					(unit 1)
+				)
+				(path "/006bc43b-d3a8-4a38-a8dc-5a24da3f9b4d/567dbb32-3fa8-4c8f-b406-7d7df1e784be/a9023d18-0b2d-43c7-9654-aa2d0b287c66"
+					(reference "C32")
 					(unit 1)
 				)
@@
 		(dnp no)
 		(fields_autoplaced yes)
-		(property "Reference" "R14"
+		(property "Reference" "R26"
 			(at 193.04 101.5999 0)
 			(effects
@@
 				(path "/006bc43b-d3a8-4a38-a8dc-5a24da3f9b4d/539d63da-e1ff-4f16-be2c-1db8c9db8078/6918b752-c4f8-49c7-b2f5-91fa140447ec"
 					(reference "R14")
+					(unit 1)
+				)
+				(path "/006bc43b-d3a8-4a38-a8dc-5a24da3f9b4d/567dbb32-3fa8-4c8f-b406-7d7df1e784be/a9023d18-0b2d-43c7-9654-aa2d0b287c66"
+					(reference "R40")
 					(unit 1)
 				)
@@
 		(dnp no)
 		(fields_autoplaced yes)
-		(property "Reference" "#PWR049"
+		(property "Reference" "#PWR070"
 			(at 111.76 55.88 0)
 			(effects
@@
 				(path "/006bc43b-d3a8-4a38-a8dc-5a24da3f9b4d/539d63da-e1ff-4f16-be2c-1db8c9db8078/6918b752-c4f8-49c7-b2f5-91fa140447ec"
 					(reference "#PWR049")
+					(unit 1)
+				)
+				(path "/006bc43b-d3a8-4a38-a8dc-5a24da3f9b4d/567dbb32-3fa8-4c8f-b406-7d7df1e784be/a9023d18-0b2d-43c7-9654-aa2d0b287c66"
+					(reference "#PWR0123")
 					(unit 1)
 				)
@@
 		(dnp no)
 		(fields_autoplaced yes)
-		(property "Reference" "C11"
+		(property "Reference" "C22"
 			(at 156.21 82.4611 90)
 			(effects
@@
 				(path "/006bc43b-d3a8-4a38-a8dc-5a24da3f9b4d/539d63da-e1ff-4f16-be2c-1db8c9db8078/6918b752-c4f8-49c7-b2f5-91fa140447ec"
 					(reference "C11")
+					(unit 1)
+				)
+				(path "/006bc43b-d3a8-4a38-a8dc-5a24da3f9b4d/567dbb32-3fa8-4c8f-b406-7d7df1e784be/a9023d18-0b2d-43c7-9654-aa2d0b287c66"
+					(reference "C34")
 					(unit 1)
 				)
@@
 		(on_board yes)
 		(dnp no)
-		(property "Reference" "C13"
+		(property "Reference" "C24"
 			(at 181.229 99.6863 0)
 			(effects
@@
 				(path "/006bc43b-d3a8-4a38-a8dc-5a24da3f9b4d/539d63da-e1ff-4f16-be2c-1db8c9db8078/6918b752-c4f8-49c7-b2f5-91fa140447ec"
 					(reference "C13")
+					(unit 1)
+				)
+				(path "/006bc43b-d3a8-4a38-a8dc-5a24da3f9b4d/567dbb32-3fa8-4c8f-b406-7d7df1e784be/a9023d18-0b2d-43c7-9654-aa2d0b287c66"
+					(reference "C36")
 					(unit 1)
 				)
@@
 		(dnp no)
 		(fields_autoplaced yes)
-		(property "Reference" "R11"
+		(property "Reference" "R23"
 			(at 120.65 91.4399 0)
 			(effects
@@
 				(path "/006bc43b-d3a8-4a38-a8dc-5a24da3f9b4d/539d63da-e1ff-4f16-be2c-1db8c9db8078/6918b752-c4f8-49c7-b2f5-91fa140447ec"
 					(reference "R11")
+					(unit 1)
+				)
+				(path "/006bc43b-d3a8-4a38-a8dc-5a24da3f9b4d/567dbb32-3fa8-4c8f-b406-7d7df1e784be/a9023d18-0b2d-43c7-9654-aa2d0b287c66"
+					(reference "R37")
 					(unit 1)
 				)
@@
 		(dnp no)
 		(fields_autoplaced yes)
-		(property "Reference" "#PWR052"
+		(property "Reference" "#PWR073"
 			(at 190.5 86.36 0)
 			(effects
@@
 				(path "/006bc43b-d3a8-4a38-a8dc-5a24da3f9b4d/539d63da-e1ff-4f16-be2c-1db8c9db8078/6918b752-c4f8-49c7-b2f5-91fa140447ec"
 					(reference "#PWR052")
+					(unit 1)
+				)
+				(path "/006bc43b-d3a8-4a38-a8dc-5a24da3f9b4d/567dbb32-3fa8-4c8f-b406-7d7df1e784be/a9023d18-0b2d-43c7-9654-aa2d0b287c66"
+					(reference "#PWR0126")
 					(unit 1)
 				)
@@
 		(on_board yes)
 		(dnp no)
-		(property "Reference" "#PWR051"
+		(property "Reference" "#PWR072"
 			(at 138.43 116.84 0)
 			(effects
@@
 				(path "/006bc43b-d3a8-4a38-a8dc-5a24da3f9b4d/539d63da-e1ff-4f16-be2c-1db8c9db8078/6918b752-c4f8-49c7-b2f5-91fa140447ec"
 					(reference "#PWR051")
+					(unit 1)
+				)
+				(path "/006bc43b-d3a8-4a38-a8dc-5a24da3f9b4d/567dbb32-3fa8-4c8f-b406-7d7df1e784be/a9023d18-0b2d-43c7-9654-aa2d0b287c66"
+					(reference "#PWR0125")
 					(unit 1)
 				)
@@
 		(dnp no)
 		(fields_autoplaced yes)
-		(property "Reference" "L1"
+		(property "Reference" "L2"
 			(at 170.18 84.1147 90)
 			(effects
@@
 				(path "/006bc43b-d3a8-4a38-a8dc-5a24da3f9b4d/539d63da-e1ff-4f16-be2c-1db8c9db8078/6918b752-c4f8-49c7-b2f5-91fa140447ec"
 					(reference "L1")
+					(unit 1)
+				)
+				(path "/006bc43b-d3a8-4a38-a8dc-5a24da3f9b4d/567dbb32-3fa8-4c8f-b406-7d7df1e784be/a9023d18-0b2d-43c7-9654-aa2d0b287c66"
+					(reference "L3")
 					(unit 1)
 				)
@@
 		(on_board yes)
 		(dnp no)
-		(property "Reference" "C10"
+		(property "Reference" "C21"
 			(at 111.379 99.6863 0)
 			(effects
@@
 				(path "/006bc43b-d3a8-4a38-a8dc-5a24da3f9b4d/539d63da-e1ff-4f16-be2c-1db8c9db8078/6918b752-c4f8-49c7-b2f5-91fa140447ec"
 					(reference "C10")
+					(unit 1)
+				)
+				(path "/006bc43b-d3a8-4a38-a8dc-5a24da3f9b4d/567dbb32-3fa8-4c8f-b406-7d7df1e784be/a9023d18-0b2d-43c7-9654-aa2d0b287c66"
+					(reference "C33")
 					(unit 1)
 				)
@@
 		(dnp no)
 		(fields_autoplaced yes)
-		(property "Reference" "D3"
+		(property "Reference" "D4"
 			(at 164.592 101.9088 90)
 			(effects
@@
 				(path "/006bc43b-d3a8-4a38-a8dc-5a24da3f9b4d/539d63da-e1ff-4f16-be2c-1db8c9db8078/6918b752-c4f8-49c7-b2f5-91fa140447ec"
 					(reference "D3")
+					(unit 1)
+				)
+				(path "/006bc43b-d3a8-4a38-a8dc-5a24da3f9b4d/567dbb32-3fa8-4c8f-b406-7d7df1e784be/a9023d18-0b2d-43c7-9654-aa2d0b287c66"
+					(reference "D6")
 					(unit 1)
 				)
@@
 		(dnp no)
 		(fields_autoplaced yes)
-		(property "Reference" "#PWR048"
+		(property "Reference" "#PWR069"
 			(at 106.68 52.07 0)
 			(effects
@@
 				(path "/006bc43b-d3a8-4a38-a8dc-5a24da3f9b4d/539d63da-e1ff-4f16-be2c-1db8c9db8078/6918b752-c4f8-49c7-b2f5-91fa140447ec"
 					(reference "#PWR048")
+					(unit 1)
+				)
+				(path "/006bc43b-d3a8-4a38-a8dc-5a24da3f9b4d/567dbb32-3fa8-4c8f-b406-7d7df1e784be/a9023d18-0b2d-43c7-9654-aa2d0b287c66"
+					(reference "#PWR0122")
 					(unit 1)
 				)
@@
 		(on_board yes)
 		(dnp no)
-		(property "Reference" "#PWR050"
+		(property "Reference" "#PWR071"
 			(at 111.76 62.23 0)
 			(effects
@@
 				(path "/006bc43b-d3a8-4a38-a8dc-5a24da3f9b4d/539d63da-e1ff-4f16-be2c-1db8c9db8078/6918b752-c4f8-49c7-b2f5-91fa140447ec"
 					(reference "#PWR050")
+					(unit 1)
+				)
+				(path "/006bc43b-d3a8-4a38-a8dc-5a24da3f9b4d/567dbb32-3fa8-4c8f-b406-7d7df1e784be/a9023d18-0b2d-43c7-9654-aa2d0b287c66"
+					(reference "#PWR0124")
 					(unit 1)
 				)
@@
 		(dnp no)
 		(fields_autoplaced yes)
-		(property "Reference" "PS1"
+		(property "Reference" "PS2"
 			(at 138.43 82.0801 0)
 			(effects
@@
 				(path "/006bc43b-d3a8-4a38-a8dc-5a24da3f9b4d/539d63da-e1ff-4f16-be2c-1db8c9db8078/6918b752-c4f8-49c7-b2f5-91fa140447ec"
 					(reference "PS1")
+					(unit 1)
+				)
+				(path "/006bc43b-d3a8-4a38-a8dc-5a24da3f9b4d/567dbb32-3fa8-4c8f-b406-7d7df1e784be/a9023d18-0b2d-43c7-9654-aa2d0b287c66"
+					(reference "PS3")
 					(unit 1)
 				)
@@
 		(on_board yes)
 		(dnp no)
-		(property "Reference" "C12"
+		(property "Reference" "C23"
 			(at 173.609 93.3363 0)
 			(effects
@@
 				(path "/006bc43b-d3a8-4a38-a8dc-5a24da3f9b4d/539d63da-e1ff-4f16-be2c-1db8c9db8078/6918b752-c4f8-49c7-b2f5-91fa140447ec"
 					(reference "C12")
+					(unit 1)
+				)
+				(path "/006bc43b-d3a8-4a38-a8dc-5a24da3f9b4d/567dbb32-3fa8-4c8f-b406-7d7df1e784be/a9023d18-0b2d-43c7-9654-aa2d0b287c66"
+					(reference "C35")
 					(unit 1)
 				)
@@
 		(dnp no)
 		(fields_autoplaced yes)
-		(property "Reference" "#PWR047"
+		(property "Reference" "#PWR068"
 			(at 100.33 85.09 0)
 			(effects
@@
 					(unit 1)
 				)
+				(path "/006bc43b-d3a8-4a38-a8dc-5a24da3f9b4d/567dbb32-3fa8-4c8f-b406-7d7df1e784be/a9023d18-0b2d-43c7-9654-aa2d0b287c66"
+					(reference "#PWR0121")
+					(unit 1)
+				)
