File: PCB_Files/layered_etu.kicad_sch (KiCad schematic)
At the start: 26 parts, among them IC5 ATTINY814-SSF, J3 Conn_01x04, M2 Motor_DC, Q5 LC191PTDT, Q6 LKPT30102B-A01, U10 Gnd, U11 GndMotor, U18 Gnd, U19 12v, U6 12v, U7 SigIn, U8 Gnd, U9 12v

Commit message: stacked version
Parts:
- removed C16, C17: 10n, Capacitor_SMD:C_0603_1608Metric, symbol Device:C
- removed C18: 1u, Capacitor_SMD:C_0603_1608Metric, symbol Device:C
- removed C19: 100n, Capacitor_SMD:C_0603_1608Metric, symbol Device:C
- removed D2: STPS5L60S, SamacSys:DIOM8059X265N, symbol SamacSys_Parts:STPS5L60S
- removed IC5: ATTINY814-SSF, SamacSys:SOIC127P600X175-14N, symbol SamacSys:ATTINY814-SSF
- removed J3: Conn_01x04, Connector_PinHeader_2.54mm:PinHeader_1x04_P2.54mm_Vertical, symbol Connector_Generic:Conn_01x04
- removed LED3: LKIR30102C-A01, SamacSys:APA3010P3C, symbol SamacSys_Parts:CSL1501RW1
- removed LED4: XL-2012IRC-940, SamacSys:LEDC2012X105N, symbol SamacSys_Parts:APTD2012SF4C
- removed M2: Motor_DC, symbol Motor:Motor_DC
- removed Q5: LC191PTDT, SamacSys:AP1608P1CP22, symbol SamacSys_Parts:AP1608P1C-P22
- removed Q6: LKPT30102B-A01, SamacSys:APA3010P3C, symbol Device:Q_Photo_NPN_CE
- removed R17, R18: 5K, Resistor_SMD:R_0603_1608Metric, symbol Device:R
- removed R19, R20: 100R, Resistor_SMD:R_0603_1608Metric, symbol Device:R
- removed R21: 10k, Resistor_SMD:R_0603_1608Metric, symbol Device:R
- removed R22: 1k, Resistor_SMD:R_0603_1608Metric, symbol Device:R
- removed U10, U18, U8: Gnd, SamacSys:Copper_Pad, symbol Copper_Pad:Copper_pad
- removed U11: GndMotor, SamacSys:Copper_Pad, symbol Copper_Pad:Copper_pad
- removed U19, U6, U9: 12v, SamacSys:Copper_Pad, symbol Copper_Pad:Copper_pad
- removed U7: SigIn, SamacSys:Copper_Pad, symbol Copper_Pad:Copper_pad
- added C46, C47: 10n, Capacitor_SMD:C_0603_1608Metric, symbol Device:C
- added C48: 1u, Capacitor_SMD:C_0603_1608Metric, symbol Device:C
- added C49: 100n, Capacitor_SMD:C_0603_1608Metric, symbol Device:C
- added D9: STPS5L60S, SamacSys:DIOM8059X265N, symbol SamacSys_Parts:STPS5L60S
- added IC10: ATTINY814-SSF, SamacSys:SOIC127P600X175-14N, symbol SamacSys:ATTINY814-SSF
- added J10, J7, J8, J9: Conn_01x01, Connector_PinHeader_2.54mm:PinHeader_1x01_P2.54mm_Vertical, symbol Connector_Generic:Conn_01x01
- added J5, J6: Conn_01x04, Connector_PinHeader_2.54mm:PinHeader_1x04_P2.54mm_Vertical, symbol Connector_Generic:Conn_01x04
- added LED7: LKIR30102C-A01, SamacSys:APA3010P3C, symbol SamacSys_Parts:CSL1501RW1
- added LED8: XL-2012IRC-940, SamacSys:LEDC2012X105N, symbol SamacSys_Parts:APTD2012SF4C
- added M4: Motor_DC, symbol Motor:Motor_DC
- added Q10: LC191PTDT, SamacSys:AP1608P1CP22, symbol SamacSys_Parts:AP1608P1C-P22
- added Q11: LKPT30102B-A01, SamacSys:APA3010P3C, symbol Device:Q_Photo_NPN_CE
- added R47, R48: 5K, Resistor_SMD:R_0603_1608Metric, symbol Device:R
- added R49, R50: 100R, Resistor_SMD:R_0603_1608Metric, symbol Device:R
- added R51: 10k, Resistor_SMD:R_0603_1608Metric, symbol Device:R
- added R52: 1k, Resistor_SMD:R_0603_1608Metric, symbol Device:R
- added TP1, TP2, TP3, TP4: TestPoint, TestPoint:TestPoint_Loop_D1.80mm_Drill1.0mm_Beaded, symbol Connector:TestPoint
- added U12: 12v, SamacSys:Copper_Pad, symbol Copper_Pad:Copper_pad
- added U16: GndMotor, SamacSys:Copper_Pad, symbol Copper_Pad:Copper_pad
- added U17: Gnd, SamacSys:Copper_Pad, symbol Copper_Pad:Copper_pad
Connections:
- net +12V: now also D9.1 (K), M4.1 (+), U12.1 (Con)
- net +3.3V: now also C48.1, C49.1, IC10.1 (VDD), J5.1 (Pin_1), J6.1 (Pin_1), J9.1 (Pin_1), R47.2, R48.2, R49.1, R50.1, R51.1
- net GND: now also C46.2, C47.2, C48.2, C49.2, IC10.14 (GND), J10.1 (Pin_1), J5.2 (Pin_2), J6.2 (Pin_2), LED7.2, LED8.1, Q10.2 (E), Q11.1 (C), U17.1 (Con)
- net updiRx: now also IC10.10 (PA0/~{RESET}/UPDI), J5.3 (Pin_3), J6.3 (Pin_3), R51.2, R52.1
- net updiTx: now also J5.4 (Pin_4), J6.4 (Pin_4), R52.2
- new net: LED7.1, R49.2
- new net: LED8.2, R50.2
- new net NMOS: IC10.3 (PA5), J7.1 (Pin_1), J8.1 (Pin_1), TP2.1
- new net Semi_Auto_In: C46.1, IC10.8 (PB1), Q10.1 (C), R48.1, TP1.1
- new net V_Cycle_In: C47.1, IC10.11 (PA1), Q11.2 (E), R47.1, TP4.1
- new net pwr_motor: D9.2 (A), M4.2 (-), U16.1 (Con)
- new net trigger_In: IC10.9 (PB0), TP3.1
Other:
- removed sheet BuckStepDown1
- removed sheet NMOSDriver2
- removed sheet TriggerDebounce1
- added sheet BuckStepDown (buck.kicad_sch)
- added sheet NMOSDriver (mos_driver.kicad_sch)
- added sheet TriggerDebounce (trigger.kicad_sch)
