File: PCB_Files/mos_driver.kicad_sch (KiCad schematic)
At the start: 6 parts, among them IC2 MCP1407-E_SN, Q3 SIR500DP-T1-RE3

Commit message: stacked version
Parts:
- C5: value 0.1u -> 1u
- C6: value 1u -> 10u
Changed lines of the file:
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@@
+					(unit 1)
+				)
+				(path "/006bc43b-d3a8-4a38-a8dc-5a24da3f9b4d/980201f8-8dc5-41cd-86ea-9e8d02f3972d/3dc01c8a-515b-4f5f-8626-294ae29ee0b9"
+					(reference "#PWR0166")
 					(unit 1)
 				)
@@
 					(unit 1)
 				)
+				(path "/006bc43b-d3a8-4a38-a8dc-5a24da3f9b4d/980201f8-8dc5-41cd-86ea-9e8d02f3972d/3dc01c8a-515b-4f5f-8626-294ae29ee0b9"
+					(reference "#PWR0167")
+					(unit 1)
+				)
 			)
 		)
@@
 					(unit 1)
 				)
+				(path "/006bc43b-d3a8-4a38-a8dc-5a24da3f9b4d/980201f8-8dc5-41cd-86ea-9e8d02f3972d/3dc01c8a-515b-4f5f-8626-294ae29ee0b9"
+					(reference "R54")
+					(unit 1)
+				)
 			)
 		)
@@
 					(unit 1)
 				)
+				(path "/006bc43b-d3a8-4a38-a8dc-5a24da3f9b4d/980201f8-8dc5-41cd-86ea-9e8d02f3972d/3dc01c8a-515b-4f5f-8626-294ae29ee0b9"
+					(reference "#PWR0172")
+					(unit 1)
+				)
 			)
 		)
@@
 				(path "/006bc43b-d3a8-4a38-a8dc-5a24da3f9b4d/783eb3f9-c065-46af-bfe5-5153fc4841ee/d346c5e5-c8a3-4b5e-a443-45f0e91c2048"
 					(reference "Q4")
+					(unit 1)
+				)
+				(path "/006bc43b-d3a8-4a38-a8dc-5a24da3f9b4d/980201f8-8dc5-41cd-86ea-9e8d02f3972d/3dc01c8a-515b-4f5f-8626-294ae29ee0b9"
+					(reference "Q12")
 					(unit 1)
 				)
@@
 					(unit 1)
 				)
+				(path "/006bc43b-d3a8-4a38-a8dc-5a24da3f9b4d/980201f8-8dc5-41cd-86ea-9e8d02f3972d/3dc01c8a-515b-4f5f-8626-294ae29ee0b9"
+					(reference "#PWR0169")
+					(unit 1)
+				)
 			)
 		)
@@
 					(unit 1)
 				)
+				(path "/006bc43b-d3a8-4a38-a8dc-5a24da3f9b4d/980201f8-8dc5-41cd-86ea-9e8d02f3972d/3dc01c8a-515b-4f5f-8626-294ae29ee0b9"
+					(reference "R53")
+					(unit 1)
+				)
 			)
 		)
@@
 					(unit 1)
 				)
+				(path "/006bc43b-d3a8-4a38-a8dc-5a24da3f9b4d/980201f8-8dc5-41cd-86ea-9e8d02f3972d/3dc01c8a-515b-4f5f-8626-294ae29ee0b9"
+					(reference "IC11")
+					(unit 1)
+				)
 			)
 		)
@@
 					(unit 1)
 				)
+				(path "/006bc43b-d3a8-4a38-a8dc-5a24da3f9b4d/980201f8-8dc5-41cd-86ea-9e8d02f3972d/3dc01c8a-515b-4f5f-8626-294ae29ee0b9"
+					(reference "#PWR0173")
+					(unit 1)
+				)
 			)
 		)
@@
 					(unit 1)
 				)
+				(path "/006bc43b-d3a8-4a38-a8dc-5a24da3f9b4d/980201f8-8dc5-41cd-86ea-9e8d02f3972d/3dc01c8a-515b-4f5f-8626-294ae29ee0b9"
+					(reference "#PWR0171")
+					(unit 1)
+				)
 			)
 		)
@@
 					(unit 1)
 				)
+				(path "/006bc43b-d3a8-4a38-a8dc-5a24da3f9b4d/980201f8-8dc5-41cd-86ea-9e8d02f3972d/3dc01c8a-515b-4f5f-8626-294ae29ee0b9"
+					(reference "#PWR0168")
+					(unit 1)
+				)
 			)
 		)
@@
 			)
 		)
-		(property "Value" "0.1u"
+		(property "Value" "1u"
 			(at 101.6 87.6299 0)
 			(effects
@@
 					(unit 1)
 				)
+				(path "/006bc43b-d3a8-4a38-a8dc-5a24da3f9b4d/980201f8-8dc5-41cd-86ea-9e8d02f3972d/3dc01c8a-515b-4f5f-8626-294ae29ee0b9"
+					(reference "C50")
+					(unit 1)
+				)
 			)
 		)
@@
 					(unit 1)
 				)
+				(path "/006bc43b-d3a8-4a38-a8dc-5a24da3f9b4d/980201f8-8dc5-41cd-86ea-9e8d02f3972d/3dc01c8a-515b-4f5f-8626-294ae29ee0b9"
+					(reference "#PWR0170")
+					(unit 1)
+				)
 			)
 		)
@@
 			)
 		)
-		(property "Value" "1u"
+		(property "Value" "10u"
 			(at 112.014 87.63 0)
 			(effects
@@
 					(unit 1)
 				)
+				(path "/006bc43b-d3a8-4a38-a8dc-5a24da3f9b4d/980201f8-8dc5-41cd-86ea-9e8d02f3972d/3dc01c8a-515b-4f5f-8626-294ae29ee0b9"
+					(reference "C51")
+					(unit 1)
+				)
